Commit message: URDF: soporte de cámara y cámara en su posición real, ToF frontal
- El soporte se apoya en el borde delantero de la placa inferior (pestaña de 3 mm) y
  sobresale ~25 mm, como en las fotos del dron.
- La cara de la tarjeta de la cámara tiene normal (0.64, 0, -0.77): el eje óptico
  apunta 50° por debajo de la horizontal (calculado de la malla del soporte).
- Nuevo tof_front_link en la parte baja del soporte, mirando al frente.

File: src/duckiedrone_dd24/urdf/dd24.urdf (robot description, URDF)
Before this commit: robot duckiedrone_dd24, 11 links, 10 joints
Links:
- added link camera_mount_link; visual mesh filename=package://duckiedrone_dd24/meshes/DD24_Camera_mount_STL.stl scale=0.001 0.001 0.001
- added link tof_front_link; visual box size=0.006 0.012 0.012
- link camera_link: geometry visual cylinder length=0.012 radius=0.007
Joints:
- added joint camera_mount_joint: type fixed, parent base_link, child camera_mount_link, origin xyz=0.093 0.01795 0 rpy=0 0 1.5708
- added joint tof_front_joint: type fixed, parent base_link, child tof_front_link, origin xyz=0.1375 0 -0.008
- joint camera_joint: origin xyz=0.075 0 0.018 -> xyz=0.1277 0 0.0082 rpy=0 0.8779 0
